File: Hardware/2LCI2C.brd (EAGLE design)
At the start: 40 x 20 mm, 37 parts, among them IC1 NAU7802-SOIC, IC2 HX711-SOP16L, IC3 TCA9548A, J3 Load Cell, J4 Load Cell, Q2 2N3906

Commit message: Partial conversion of early concept PCB.
Parts:
- removed C12, C4: 10uF, SuperHouse-DiscreteSemi:C0805
- removed C5: 100nF, SuperHouse-DiscreteSemi:C0603
- removed Q2: 2N3906, SuperHouse-DiscreteSemi:SOT23-BEC
- removed R13: 10K, SuperHouse-DiscreteSemi:R0603
- removed R14: 8K2, SuperHouse-DiscreteSemi:R0603
- added R11, R2: 10K, SuperHouse-DiscreteSemi:R0603
- IC2: value HX711-SOP16L -> NAU7802-SOIC; device SuperHouse-ICs:SOP16-L -> SuperHouse-ICs:SO16
- J3: value Load Cell -> X Load Cell
- J4: value Load Cell -> Y Load Cell
- R10, R9: value 100R -> 47R
- R5: value 8K2 -> 10K
- moved R5 34.9 mm to (2.00, -9.00), turned to 0 degrees
- moved C13 32.4 mm to (29.0, 8.00)
- moved R4 32.2 mm to (2.00, -6.00), turned to 0 degrees
- moved IC3 18.5 mm to (5.90, 13.1), turned to 180 degrees
- moved IC1 13.0 mm to (20.0, 13.0), turned to 180 degrees
- moved IC2 13.0 mm to (33.0, 13.0), turned to 0 degrees
- turned R1 to 270 degrees
- turned R10 to 270 degrees
- turned R3 to 270 degrees
- turned R9 to 270 degrees
Connections:
- removed net MOSI_SDA: J2.2, R8.1
- removed net N$14: C9.1, IC2.7, R9.2
- removed net N$15: C9.2, IC2.8, R10.2
- removed net N$16: IC2.3, Q2.C, R13.2
- removed net N$17: C8.1, IC2.6
- removed net N$20: IC2.2, Q2.B
- removed net N$21: IC2.4, R13.1, R14.2
- removed net PA0: IC2.12
- removed net PA1: IC2.11
- removed net SCK_SCL: J2.3, R7.1
- removed net X_E+: C10.1, C11.1, J3.1
- new net N$6: C9.1, IC1.2, R9.1
- new net N$7: C9.2, IC1.3, R10.1
- new net N$9: C10.1, C11.1, IC1.1, IC1.16
- new net SCL0: IC1.13, IC3.5, R11.1
- new net SCL1: IC2.13, IC3.7, R2.1
- new net SDA0: IC1.14, IC3.4, R5.1
- new net SDA1: IC2.14, IC3.6, R4.1
- new net X_B+: IC1.5, J3.1
- new net X_B-: IC1.4, J3.2
- net GND: now also IC2.7, IC2.8, IC2.9, IC3.12; no longer C12.2, IC2.14, IC2.5, J3.2, R14.1
- net N$1: now also IC2.6; no longer IC1.6
- net N$2: now also IC2.2, R1.1; no longer IC1.2, R1.2
- net N$3: now also IC2.1, IC2.16; no longer IC1.1, IC1.16
- net N$4: now also IC2.3, R3.1; no longer IC1.3, R3.2
- net N$8: now also C8.1, IC1.6; no longer IC2.13
- net SCL: now also IC3.22, J2.3, R7.1; no longer IC1.13
- net SDA: now also IC3.23, J2.2, R8.1; no longer IC1.14
- net VCC: now also IC3.24, R11.2, R2.2, R4.2, R5.2; no longer C12.1, IC2.1, IC2.15, IC2.16, Q2.E
- net X_A+: now also R10.2; no longer R10.1
- net X_A-: now also R9.2; no longer R9.1
- net Y_A+: now also R3.2; no longer R3.1
- net Y_A-: now also R1.2; no longer R1.1
- net Y_B+: now also IC2.5; no longer IC1.5
- net Y_B-: now also IC2.4; no longer IC1.4
Routing:
- net PA0: track 19.0 -> 0.00 mm, vias 1 -> 0
- net PA1: track 18.7 -> 0.00 mm, vias 1 -> 0
- net SCL: track 0.00 -> 18.5 mm
- net SCK_SCL: track 18.5 -> 0.00 mm
- net VCC: track 14.3 -> 1.65 mm, vias 2 -> 1
- net SDA: track 0.00 -> 12.2 mm
- net MOSI_SDA: track 12.2 -> 0.00 mm
- net N$14: track 8.39 -> 0.00 mm
- net N$16: track 8.15 -> 0.00 mm
- net N$15: track 4.65 -> 0.00 mm
- net N$21: track 4.00 -> 0.00 mm
- net X_E+: track 3.11 -> 0.00 mm
- net N$17: track 2.71 -> 0.00 mm
- net N$20: track 2.56 -> 0.00 mm
- net X_A+: track 1.79 -> 0.00 mm
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