File: Hardware/ZSLC.brd (EAGLE design)
At the start: 23 x 19 mm, 22 parts, among them IC1 NAU7802-SOIC, J1 I2C, J22 DRDY, J3 X Load Cell, J4 Y Load Cell

Commit message: Fixed labels and values on X and Y axis connectors.
Parts:
- J3: value X Load Cell -> Y Load Cell
- J4: value Y Load Cell -> X Load Cell
Changed lines of the file:
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@@
 <layer number="19" name="Unrouted" color="12" fill="1" visible="yes" active="yes"/>
 <layer number="20" name="Dimension" color="15" fill="1" visible="yes" active="yes"/>
-<layer number="21" name="tPlace" color="15" fill="1" visible="no" active="yes"/>
-<layer number="22" name="bPlace" color="14" fill="1" visible="yes" active="yes"/>
+<layer number="21" name="tPlace" color="15" fill="1" visible="yes" active="yes"/>
+<layer number="22" name="bPlace" color="14" fill="1" visible="no" active="yes"/>
 <layer number="23" name="tOrigins" color="15" fill="1" visible="yes" active="yes"/>
 <layer number="24" name="bOrigins" color="15" fill="1" visible="yes" active="yes"/>
@@
 <attribute name="VALUE" x="1.484" y="17.1348" size="0.8128" layer="27" font="vector"/>
 </element>
-<element name="J3" library="SuperHouse-Connectors" library_urn="urn:adsk.eagle:library:11765989" package="1X04-1.27-PLAIN" package3d_urn="urn:adsk.eagle:package:19968944/2" value="X Load Cell" x="20" y="4" smashed="yes" rot="R90">
+<element name="J3" library="SuperHouse-Connectors" library_urn="urn:adsk.eagle:library:11765989" package="1X04-1.27-PLAIN" package3d_urn="urn:adsk.eagle:package:19968944/2" value="Y Load Cell" x="20" y="4" smashed="yes" rot="R90">
 <attribute name="NAME" x="19.135" y="4" size="1.27" layer="25" font="vector" ratio="10" rot="R90" align="bottom-center"/>
 <attribute name="VALUE" x="21.165" y="4" size="0.8128" layer="27" font="vector" ratio="16" rot="R90" align="top-center"/>
 </element>
-<element name="J4" library="SuperHouse-Connectors" library_urn="urn:adsk.eagle:library:11765989" package="1X04-1.27-PLAIN" package3d_urn="urn:adsk.eagle:package:19968944/2" value="Y Load Cell" x="20" y="11" smashed="yes" rot="R90">
+<element name="J4" library="SuperHouse-Connectors" library_urn="urn:adsk.eagle:library:11765989" package="1X04-1.27-PLAIN" package3d_urn="urn:adsk.eagle:package:19968944/2" value="X Load Cell" x="20" y="11" smashed="yes" rot="R90">
 <attribute name="NAME" x="19.135" y="11" size="1.27" layer="25" font="vector" ratio="10" rot="R90" align="bottom-center"/>
 <attribute name="VALUE" x="21.165" y="11" size="0.8128" layer="27" font="vector" ratio="16" rot="R90" align="top-center"/>
